File: ESP32_DevKit.kicad_sch (KiCad schematic)
At the start: 34 parts, among them IC1 CP2102N-A01-GQFN28, J1 USB_B_Micro, J2 Conn_01x19_Male, J3 Conn_01x19_Male, Q1 MMSS8050-H-TP, Q2 MMSS8050-H-TP, SW1 SW_Push, SW2 SW_Push, U1 AMS1117-3.3

Commit message: PCB design completed
Parts:
- C1, C2, C3, C4, C5, C6, C7, C8, C9: footprint (none) -> Capacitor_SMD:C_0805_2012Metric_Pad1.18x1.45mm_HandSolder
- D1: footprint (none) -> LED_SMD:LED_0805_2012Metric_Pad1.15x1.40mm_HandSolder
- D2, D3, D4: value LESD5D5.0CtT1G -> LESD5D5.0CT1G; footprint (none) -> LESD5D5:SODFL1608X70N
- D5: footprint (none) -> BAT760-7:SOD2513X120N
- J1: footprint (none) -> Connector_USB:USB_Micro-AB_Molex_47590-0001
- J2, J3: footprint (none) -> Connector_PinHeader_2.54mm:PinHeader_1x19_P2.54mm_Vertical
- R1, R10, R2, R3, R4, R5, R6, R7, R8, R9: footprint (none) -> Resistor_SMD:R_0805_2012Metric_Pad1.20x1.40mm_HandSolder
- SW1, SW2: footprint (none) -> Button_Switch_SMD:SW_Push_1P1T_NO_6x6mm_H9.5mm
